File: project-alpha/project-alpha.sch (EAGLE design)
At the start: 0 parts

Commit message: Schematic entry for most parts of project alpha
Design has WiFi module, I2C EEPROM, LDO, LED, SD card, and matching
circuit for antenna.  The antenna isn't included yet as that part
still needs to be created in the library (going with the ACX reference
design part).

Also included solder jumper pads for end user customizations for I2C
EEPROM address, SD card chip select and CC3000 chip select.  These will
be on the back side of the board for easy customization and rewiring.
The user would need to cut the thin trace (10mil) and then resolder to
the pin they want to use (as well as change the software accordingly).

Signed-off-by: fangsuei <fangsuei@fangsuei.com>
Parts:
- added ANAPORT: (no value), pinhead:PINHD-1X6
- added C1: (no value), resistor:C-EUC0402
- added C2: (no value), rcl:C-EUC0402
- added DIGHIPORT: (no value), pinhead:PINHD-1X10
- added DIGLOPORT, PWRPORT: (no value), pinhead:PINHD-1X8
- added L1, L2: (no value), microbuilder:INDUCTOR_0402
- added LED1: (no value), microbuilder:LED0603_NOOUTLINE
- added R1, R2: 0, resistor:R-EU_R0402
- added SJ1, SJ2, SJ3, SJ4, SJ5, SJ6: (no value), microbuilder:SOLDERJUMPER_CLOSED
- added TPRX, TPTX: (no value), microbuilder:TESTPOINT
- added U$2: MICROSD, adafruit:MICROSD
- added U1: CC3000-MOD, eightbitlabs:CC3000-MOD
- added U2: TLV1117-33, eightbitlabs:TLV1117-33
- added U3: TXS0108E, eightbitlabs:TXS0108E
- added U4: 24AA512, eightbitlabs:24AA512
Connections:
- new net +3V3: PWRPORT.4, R1.1, R2.1, U$2.VDD, U1.VIO_HOST, U2.OUT, U3.VCCA
- new net +5V: U3.OE, U3.VCCB, U4.VCC
- new net GND: L1.1, L2.1, PWRPORT.6, PWRPORT.7, SJ4.1, SJ5.1, SJ6.1, U$2.GND, U$2.GND1, U$2.VSS, U1.GND, U2.GND, U3.GND, U4.VSS, U4.WP
- new net N$1: PWRPORT.5, U2.IN
- new net N$10: C1.1, C2.1, L1.2
- new net N$11: DIGHIPORT.6, U3.B4
- new net N$12: U1.SCL_EEPROM, U1.SDA_EEPROM
- new net N$13: U1.SCL_CC3000, U1.SDA_CC3000
- new net N$14: DIGHIPORT.7, U3.B3
- new net N$15: DIGHIPORT.5, U3.B2
- new net N$16: U$2.CS, U3.A7
- new net N$17: SJ1.1, U3.B1
- new net N$18: DIGHIPORT.8, SJ1.2
- new net N$19: SJ2.1, U3.B7
- new net N$2: U1.SPI_CS, U3.A1
- new net N$20: DIGLOPORT.4, SJ2.2
- new net N$21: LED1.A, R2.2
- new net N$22: LED1.C, SJ3.1
- new net N$23: DIGLOPORT.5, SJ3.2
- new net N$24: SJ4.2, U4.A0
- new net N$25: SJ5.2, U4.A1
- new net N$26: SJ6.2, U4.A2
- new net N$27: DIGHIPORT.1, U4.SCL
- new net N$28: DIGHIPORT.2, U4.SDA
- new net N$29: C2.2, L2.2
- new net N$3: U$2.SCLK, U1.SPI_CLK, U3.A2
- new net N$30: TPTX.P$1, U1.WL_RS232_TX
- new net N$31: TPRX.P$1, U1.WL_RS232_RX
- new net N$4: U$2.DATA_IN, U1.SPI_DIN, U3.A3
- new net N$5: U$2.DATA_OUT, U1.SPI_DOUT, U3.A4
- new net N$6: U1.SPI_IRQ, U3.A5
- new net N$7: U1.VBAT_SW_EN, U3.A6
- new net N$8: C1.2, U1.RF_ANT
- new net N$9: R1.2, U1.VBAT_IN
